File: Frequency_Counter_FPGA_Module/FPGA_Module_2_0/FPGA_module.kicad_pcb (KiCad board)
At the start: 4 copper layers, 98 x 89 mm, 283 parts, among them IC1 74HC390D, J1 Channel A, J10 OCXO_TTL, J12 GPS_CLK, J13 OCXO_DIV, J14 PLL2_CLK2, J15 PLL2_CLK1, J16 10MHz TTL, J17 10MHz TTL, J18 10MHz TTL, J19 10MHz TTL, J2 Channel B, J3 CH A Test, J4 CH B Test, J5 GPS, J6 Input_board, J7 STM_mainboard, J8 OCXO_VC, J9 OCXO_OPA, U1 MAX9601, U10 TS5A3159DCK, U11 MIC920, U12 TLV9001IDCK, U13 OPA365DBV, U14 74LVC1G86, U15 LMK1C1104, U16 LMR33630ADDAR, U17 B0505S-1W, U18 LMR33630ADDAR, U19 LMK1C1104, U2 MC100EP016A, U20 MC100EPT23DT, U21 OPA365DBV, U22 74LVC1G17, U23 74LVC1G17, U24 MC100EPT23DT, U4 SI5356A, U5 ADS1115, U6 TMP117xxDRV, U8 TMP117xxDRV

Commit message: feat(boot): LED selftest blikaci kod + RTC LSE medium-low drive; UI 4.3" audit; FPGA HW revize
STM32H757 firmware:
- bootled.c/h: boot-time HW selftest diagnostika na LED_1 (PG3). Kazdy
  sledovany periferni init (FMC/SPI2/I2C4/DSIHOST/LTDC/USART1/RTC/ADC3/
  QUADSPI/I2C1) + display bring-up (panel probe/power-on/DSI start/
  TC358762) si zaznamena poradove cislo; pri zaseknuti v Error_Handler()
  LED bez displeje zabliká N-krat podle poradi. Regen-safe (jen chranene
  USER CODE hooky), bez zpozdeni v happy-path.
- RTC LSE Drive Capability LOW -> MEDIUM LOW (H757_LED.ioc): kompenzuje
  desky s predimenzovanymi zatezovymi kondenzatory krystalu (22pF misto
  18pF), ktere LSE nerozjizdely.
- UI audit pro realny 4,3" 800x480 panel (8,54 px/mm): hit-slop pilulek,
  fonty, HDR_PILL_LIMIT fit-check, Menu 3x4 mrizka s placeholdery, oprava
  ghost bugu AUTO CET/CEST tlacitka, sign-loss bug ve fmt_fixed/fmt_minmax.
  main-old layout zamrazen jako default (A/B srovnani, viz STATUS.md #14).

FPGA carrier v2.0 (KiCad): prubezne review checklisty a schema/PCB revize.

Co-Authored-By: OK2JNJ <ok2jnj@local>
Parts:
- removed C120: 100n, Capacitor_SMD:C_0805_2012Metric
- removed the C48 at (90.6, 119.8)
- removed the C65 at (76.0, 120.2)
- removed the C66 at (66.8, 123.6)
- removed the C67 at (73.8, 122.2)
- removed IC1: 74HC390D, Package_SO:SOIC-16_3.9x9.9mm_P1.27mm
- removed the J12 at (74.7, 126.5)
- removed the J3 at (75.0, 92.5)
- removed the J4 at (75.0, 74.3)
- removed the J8 at (88.0, 133.9)
- removed JP2: PLL_FREQ, Jumper:SolderJumper-3_P1.3mm_Open_RoundedPad1.0x1.5mm_NumberLabels
- removed R107, R110, R111, R112: 33R, Resistor_SMD:R_0805_2012Metric
- removed R108: 10k0, Resistor_SMD:R_0805_2012Metric
- removed R109: 100k, Resistor_SMD:R_0805_2012Metric
- removed the R51 at (102.8, 129.1)
- removed the R57 at (92.8, 128.8)
- removed the R58 at (88.4, 119.7)
- removed the R60 at (85.5, 118.8)
- removed the R65 at (66.8, 125.5)
- removed the R66 at (71.0, 122.9)
- removed the U14 at (72.1, 119.3)
- removed the U2 at (82.8, 83.7)
- added C32: 100n, Capacitor_SMD:C_0805_2012Metric, F.Cu at (48.7, 47.1)
- added C33: 100p, Capacitor_SMD:C_0805_2012Metric, F.Cu at (48.7, 50.1)
- added C53: 100n, Capacitor_SMD:C_0805_2012Metric, F.Cu at (35.0, 36.1)
- added C55: 100n, Capacitor_SMD:C_0805_2012Metric, F.Cu at (-3.62, 70.4)
- added C56: 10n, Capacitor_SMD:C_0805_2012Metric, F.Cu at (35.0, 45.1)
- added C59: 100n, Capacitor_SMD:C_0805_2012Metric, F.Cu at (48.7, 36.1)
- added C70: 10n, Capacitor_SMD:C_0805_2012Metric, F.Cu at (-15.0, 57.0)
- added C73: 100n, Capacitor_SMD:C_0805_2012Metric, F.Cu at (-15.0, 60.0)
- added C74: 1n, Capacitor_SMD:C_0805_2012Metric, F.Cu at (-15.0, 63.0)
- added C78: 10n, Capacitor_SMD:C_0805_2012Metric, F.Cu at (48.7, 42.1)
- added R48: 10k, Resistor_SMD:R_0805_2012Metric, F.Cu at (53.1, 50.0)
- added R72: 82R, Resistor_SMD:R_0805_2012Metric, F.Cu at (53.1, 40.9)
- added R73: 4k7, Resistor_SMD:R_0805_2012Metric, F.Cu at (-19.4, 57.0)
- added R79: 49R9, Resistor_SMD:R_0805_2012Metric, F.Cu at (-19.4, 59.9)
- added R80: 5k6, Resistor_SMD:R_0805_2012Metric, F.Cu at (-19.4, 62.9)
- added R81: 10k0, Potentiometer_SMD:Potentiometer_Bourns_3224W_Vertical, F.Cu at (-14.0, 67.6)
- added R82: 33k, Resistor_SMD:R_0805_2012Metric, F.Cu at (-19.4, 65.8)
- added R84: 12k, Resistor_SMD:R_0805_2012Metric, F.Cu at (-19.4, 68.8)
- added R85: 12k, Resistor_SMD:R_0805_2012Metric, F.Cu at (-19.4, 71.7)
- added U12: AD5693RxRM, Package_SO:MSOP-10_3x3mm_P0.5mm, F.Cu at (40.8, 36.9)
- added U18: MIC920, Package_TO_SOT_SMD:SOT-353_SC-70-5, F.Cu at (-10.8, 61.8)
- added U3: MC100EP016A, Package_QFP:LQFP-32_7x7mm_P0.8mm, F.Cu at (82.6, 85.9)
- added U7: 74LVC1G17, Package_TO_SOT_SMD:SOT-23-5, F.Cu at (36.6, 105.3)
- C1: renamed from C58; moved to B.Cu
- C2: renamed from C59; moved to B.Cu
- C24: renamed from C106; moved to B.Cu
- C29: renamed from C107; moved to B.Cu
- C3: renamed from C63; moved to B.Cu
- C30: renamed from C108; moved to B.Cu
- C4: renamed from C109; moved to B.Cu
- C5: renamed from C112; moved to B.Cu
- C50: renamed from C45; moved to B.Cu
- C54: moved to F.Cu
- C6: renamed from C113; moved to B.Cu
- C68: renamed from C60; value 100u -> 1u
- C79: renamed from C71; moved to B.Cu
- D2: value BAR64 -> BAT54S; footprint Diode_SMD:D_SOD-523 -> Package_TO_SOT_SMD:SOT-23; moved to F.Cu
- J10: value OCXO_TTL -> REF_Test
- J6: renamed from J14; value PLL2_CLK2 -> CLK_OUT_1
- J7: renamed from J15; value PLL2_CLK1 -> CLK_OUT_2
- J9: renamed from J13; value OCXO_DIV -> Ext. Ref.
- R33: renamed from R22; moved to B.Cu
- R50: value 1k0 -> 33R
- R78: renamed from R63; value 100k -> 47k
- R86: renamed from R88; moved to B.Cu
- U17: renamed from U22; moved to B.Cu
- moved R7 124.6 mm to (62.7, 95.1), turned to 180 degrees
- moved U17 114.7 mm to (73.8, 106.3), turned to 180 degrees
- moved R10 113.7 mm to (69.1, 72.8)
- moved D2 103.1 mm to (-10.3, 57.7), turned to 0 degrees
- moved R86 101.1 mm to (69.2, 107.5), turned to 180 degrees
- moved R50 97.9 mm to (53.1, 47.1), turned to 0 degrees
- moved C79 91.2 mm to (69.0, 105.3)
- moved C54 78.4 mm to (35.0, 39.1), turned to 0 degrees
- moved R44 67.1 mm to (93.8, 93.3), turned to -90 degrees
- moved R45 65.9 mm to (93.8, 85.8), turned to 90 degrees
- moved R40 65.2 mm to (90.9, 94.5), turned to 180 degrees
- moved C45 63.8 mm to (107.7, 93.2), turned to -90 degrees
- moved C61 62.3 mm to (35.2, 141.5)
- moved R33 62.0 mm to (86.5, 94.7)
- moved C28 60.7 mm to (95.8, 85.8), turned to -90 degrees
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- renumbered C79 to C100, C93 to C101, C80 to C102, C81 to C103, C94 to C104, C82 to C105, C95 to C106, C83 to C107, C96 to C108, C84 to C109, C85 to C110, C97 to C111, C87 to C112, C98 to C113, C86 to C114, C88 to C115, C89 to C116, C99 to C117, C90 to C118, C110 to C19, C111 to C20, C19 to C21, C20 to C22, C21 to C23, C22 to C25, C50 to C26, C64 to C27, C57 to C28, C23 to C31, C24 to C34, C25 to C35, C26 to C36, C27 to C37, C28 to C38, C29 to C39, C33 to C40, C34 to C41, C30 to C42, C31 to C43, C32 to C44, C114 to C45, C35 to C46, C36 to C47, C37 to C48, C38 to C49, C4 to C51, C5 to C52, C46 to C57, C47 to C58, C49 to C60, C51 to C61, C103 to C62, C104 to C63, C52 to C64, C53 to C65, C55 to C66, C56 to C67, C6 to C69, C61 to C71, C105 to C72, C62 to C75, C118 to C76, C119 to C77, C116 to C80, C1 to C81, C2 to C82, C117 to C83, C68 to C84, C69 to C85, C3 to C86, C70 to C87, C72 to C88, C76 to C89, C73 to C90, C100 to C91, C101 to C92, C74 to C93, C102 to C94, C75 to C95, C77 to C96, C91 to C97, C78 to C98, C92 to C99, D5 to D4, D4 to D5, F3 to F2, F2 to F3, FB3 to FB2, FB2 to FB3, J16 to J11, J17 to J12, J18 to J13, J19 to J14, J5 to J3, J6 to J4, J7 to J5, J9 to J8, L3 to L1, L6 to L2, L4 to L3, L5 to L4, L7 to L5, R85 to R10, R79 to R100, R76 to R101, R80 to R102, R77 to R103, R9 to R11, R10 to R12, R11 to R13, R12 to R14, R13 to R15, R14 to R16, R23 to R17, R24 to R18, R104 to R19, R16 to R20, R15 to R22, R105 to R23, R18 to R24, R103 to R25, R17 to R26, R19 to R27, R20 to R28, R64 to R29, R25 to R30, R33 to R31, R26 to R32, R27 to R34, R99 to R35, R28 to R36, R100 to R37, R34 to R38, R59 to R39, R61 to R40, R31 to R41, R102 to R42, R32 to R43, R62 to R44, R101 to R45, R29 to R46, R30 to R47, R113 to R49, R96 to R51, R92 to R52, R89 to R53, R90 to R54, R97 to R55, R98 to R56, R37 to R57, R38 to R58, R39 to R59, R40 to R60, R41 to R61, R42 to R62, R43 to R63, R44 to R64, R45 to R65, R35 to R66, R36 to R67, R52 to R68, R53 to R69, R86 to R7, R71 to R70, R72 to R71, R54 to R74, R81 to R75, R55 to R76, R87 to R77, R7 to R8, R106 to R83, R56 to R87, R82 to R88, R83 to R89, R8 to R9, R84 to R90, R67 to R91, R68 to R92, R69 to R93, R70 to R94, R73 to R95, R48 to R96, R74 to R97, R75 to R98, R78 to R99, U6 to U10, U8 to U11, U9 to U13, U21 to U14, U13 to U15, U11 to U16, U10 to U19, U24 to U2, U23 to U20, U15 to U21, U19 to U22, U16 to U23, U18 to U24, U17 to U25, U12 to U4, U20 to U5, U3 to U6, U5 to U8, U4 to U9
Connections:
- net /FPGA_core/GPS_CLK_OUT renamed GPS_CLK_Out
- net /GPSDO/10MHz_GPSDO_CLK2 renamed 10MHz_GPSDO_CLK2
- net GPS_Time_Stamp renamed GPS_Ext_Int
- C54 pad 1: GND -> +5V
- C54 pad 2: +5V -> GND
- C61 pad 2: Net-(C51-Pad2) -> Net-(C61-Pad2)
- C88 pad 1: /FPGA_core/10MHz_GPSDO_CLK4 -> unconnected-(C88-Pad1)
- C90 pad 1: /GPSDO/10MHz_GPSDO_CLK3 -> /FPGA_core/10MHz_GPSDO_CLK3
- D2 pad 1: Net-(D2-K) -> GND
- D2 pad 2: Net-(D2-A) -> +3V3
- J4 pad 6: Input_Mod_CS1 -> unconnected-(J4-Pin_6-Pad6)
- J4 pad 7: unconnected-(J6-Pin_7-Pad7) -> Input_Mod_CS1
- J5 pad 6: Input_Mod_CS1 -> FPGA_CS2
- J5 pad 7: FPGA_CS2 -> Input_Mod_CS1
- J9 pad 1: Net-(J13-In) (its old number) -> Net-(D2-COM)
- R50 pad 1: Net-(R51-A) -> GPS_CLK_Buff
- R50 pad 2: +5V -> Net-(U6-PIN31_IOB15A_RGBINIT)
- R51 pad 2: /GPSDO/OCXO_VC -> /GPSDO/OCXO_VC_Sense
- R62 pad 1: /GPSDO/10MHz_GPSDO_CLK3 -> /GPSDO/10MHz_GPSDO_CLK1
- R70 pad 1: /I2C_devices/PLL2_CLK2 -> CLK_OUT_1
- R71 pad 1: /I2C_devices/PLL2_CLK1 -> CLK_OUT_2
- R78 pad 2: Net-(R63-Pad2) -> /GPSDO/OCXO_VC
- R83 pad 1: Net-(C67-Pad1) -> Net-(R83-Pad1)
- R83 pad 2: Net-(R106-Pad2) -> Net-(R83-Pad2)
- R86 pad 1: Net-(R88-Pad1) -> Net-(R86-Pad1)
- R89 pad 2: /GPSDO/10MHz_GPSDO_CLK3 -> /FPGA_core/10MHz_GPSDO_CLK3
- R90 pad 2: /FPGA_core/10MHz_GPSDO_CLK4 -> unconnected-(C88-Pad1)
- U13 pad 1: Net-(U21-+) -> Net-(U13-VC)
- U14 pad 1: /GPSDO/OCXO_VC -> /GPSDO/OCXO_VC_Sense
- U14 pad 3: Net-(U21-+) -> Net-(U13-VC)
- U14 pad 4: /GPSDO/OCXO_VC -> /GPSDO/OCXO_VC_Sense
- U15 pad 1: Net-(R57-Pad2) -> Net-(U15--)
- U15 pad 4: Net-(U13--) -> Net-(U15--)
- U17 pad 4: Net-(R88-Pad1) -> Net-(R83-Pad1)
- U19 pad 1: Net-(C51-Pad2) -> Net-(U19-Pad1)
- U19 pad 3: Net-(R51-S) -> Net-(R83-Pad2)
- U19 pad 4: Net-(U21-+) -> Net-(R86-Pad1)
- U19 pad 6: OCXO_VC_SW -> /FPGA_core/Ref_Ctrl
- U20 pad 4: OCXO_VC_SW -> Net-(U19-Pad1)
- U6 pad 11: /FPGA_core/PLL_CLK4 -> /FPGA_core/PLL_CLK2
- U6 pad 12: /FPGA_core/PLL_CLK2 -> unconnected-(U6-PIN34_IOB23B_RGB_VS-Pad12)
- U6 pad 15: unconnected-(U3-PIN41_IOB41A_RGB_B7-Pad15) -> DIV_Bit1/2
- U6 pad 17: DIV_Out -> /FPGA_core/Ref_Ctrl
- U6 pad 18: DIV_Res -> unconnected-(U6-PIN53_IOR15B_RGB_B4-Pad18)
- U6 pad 28: unconnected-(U3-PIN31_IOB15A_RGBINIT-Pad28) -> Net-(U6-PIN31_IOB15A_RGBINIT)
- U6 pad 29: unconnected-(U3-PIN49_IOR24A_SPILCD_RS-Pad29) -> Reset
- U6 pad 38: /FPGA_core/PLL_INT -> unconnected-(U6-PIN76_IOT37B_SPILCD_MCLK-Pad38)
- U6 pad 39: Reset -> unconnected-(U6-PIN77_IOT37A_SPILCD_MO-Pad39)
- U6 pad 48: /FPGA_core/10MHz_GPSDO_CLK4 -> /FPGA_core/10MHz_GPSDO_CLK3
- U6 pad 7: DIV_Bit3/4 -> unconnected-(U6-PIN27_IOB11A-Pad7)
- U6 pad 8: DIV_Bit1/2 -> DIV_Bit3/4
- U6 pad 9: unconnected-(U3-PIN29_IOB13A-Pad9) -> /FPGA_core/PLL_CLK4
- U9 pad 13: Net-(U4-CLK_5) -> CLK_OUT_1
- U9 pad 9: Net-(U4-CLK_7) -> CLK_OUT_2
Routing:
- net +3V3: track 492.2 -> 29.9 mm, vias 35 -> 5
- net GND: track 273.3 -> 78.0 mm, vias 381 -> 260
- net /FPGA_core/SDA: track 189.5 -> 0.00 mm, vias 7 -> 0
- net /FPGA_core/SCL: track 188.0 -> 0.00 mm, vias 7 -> 0
- net +5V: track 146.5 -> 20.6 mm, vias 4 -> 2
- net unconnected-(J4-Pin_9-Pad9): track 117.5 -> 0.00 mm, vias 1 -> 0
- net /FPGA_core/PLL_INT: track 112.3 -> 1.91 mm, vias 5 -> 0
- net Reset: track 117.9 -> 26.1 mm, vias 3 -> 2
- net GPS_CLK_Out: track 49.2 -> 0.00 mm
- net +12V: track 49.9 -> 1.27 mm, vias 5 -> 0
- net /GPSDO/10MHz_GPSDO_CLK3: track 43.1 -> 0.00 mm, vias 2 -> 0
- net OCXO_VC_SW: track 34.4 -> 0.00 mm, vias 2 -> 0
- net Net-(U8-AIN2): track 31.6 -> 0.00 mm, vias 2 -> 0
- net /I2C_devices/PLL2_CLK2: track 31.5 -> 0.00 mm, vias 1 -> 0
- net /I2C_devices/PLL2_CLK1: track 29.6 -> 0.00 mm, vias 3 -> 0
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